Commit message: feat:增加调试修改文件

File: src/hunter_bipedal_control/legged_examples/legged_hunter/legged_hunter_description/urdf/hunter.urdf (robot description, URDF)
Before this commit: robot hunter, 16 links, 15 joints
Links:
- link base_link: mass 5.673631 -> 9.2349183; geometry collision box size=0.001 0.001 0.001; visual mesh filename=package://legged_hunter_description/tangba_meshes/base_link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
- link leg_l1_link: mass 0.453728 -> 1.2581230; geometry collision box size=0.001 0.001 0.001; visual mesh filename=package://legged_hunter_description/tangba_meshes/link_left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
- link leg_l2_link: mass 0.925998 -> 0.4307105; geometry collision box size=0.001 0.001 0.001; visual mesh filename=package://legged_hunter_description/tangba_meshes/link_left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
- link leg_l3_link: mass 1.390468 -> 2.9774665; geometry collision box size=0.001 0.001 0.001; visual mesh filename=package://legged_hunter_description/tangba_meshes/link_left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
- link leg_l4_link: mass 0.649518 -> 1.5242262; geometry collision box size=0.001 0.001 0.001; visual mesh filename=package://legged_hunter_description/tangba_meshes/link_left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
- link leg_l5_link: mass 0.030265 -> 1.3694143; geometry collision box size=0.001 0.001 0.001; visual mesh filename=package://legged_hunter_description/tangba_meshes/link_left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
- link leg_l_f1_link: mass 0.01 -> None; geometry 
- link leg_l_f2_link: mass 0.01 -> None; geometry 
- link leg_r1_link: mass 0.453728 -> 1.2581230; geometry collision box size=0.001 0.001 0.001; visual mesh filename=package://legged_hunter_description/tangba_meshes/link_righ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
- link leg_r2_link: mass 0.925998 -> 0.4307105; geometry collision box size=0.001 0.001 0.001; visual mesh filename=package://legged_hunter_description/tangba_meshes/link_righ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
- link leg_r3_link: mass 1.388625 -> 2.9802188; geometry collision box size=0.001 0.001 0.001; visual mesh filename=package://legged_hunter_description/tangba_meshes/link_righ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
- link leg_r4_link: mass 0.614720 -> 1.5250154; geometry collision box size=0.001 0.001 0.001; visual mesh filename=package://legged_hunter_description/tangba_meshes/link_righ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
- link leg_r5_link: mass 0.030265 -> 1.3695979; geometry collision box size=0.001 0.001 0.001; visual mesh filename=package://legged_hunter_description/tangba_meshes/link_righ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
- link leg_r_f1_link: mass 0.01 -> None; geometry 
- link leg_r_f2_link: mass 0.01 -> None; geometry 
Joints:
- joint leg_l1_joint: axis 1 0 0 -> 0 0 1; limit lower=-0.2 upper=0.5 effort=23.7 velocity=30.1 -> lower=-0.34906 upper=0.34906 effort=12 velocity=14; origin xyz=-0.002 0.09 -0.1035 rpy=0 0 0 -> xyz=0.0200750000000063 0.0680000000000003 0.138 rpy=0 0 0
- joint leg_l2_joint: axis 0 0 1 -> -0.0355014772726285 0 0.999369623868697; limit lower=-0.5 upper=1 effort=23.7 velocity=30.1 -> lower=-0.1745 upper=0.34906 effort=12 velocity=14; origin xyz=0 -0.00016972 -0.0325 rpy=0 0 0 -> xyz=0.0225 0 -0.0715 rpy=-1.5707963267949 0 1.57079632679489
- joint leg_l3_joint: axis 0 -1 0 -> 0.0355014772726165 0 0.999369623868697; limit lower=-0.8 upper=1.2 effort=23.7 velocity=30.1 -> lower=-0.6981 upper=1.8 effort=12 velocity=14; origin xyz=0 -0.01433 -0.0575 rpy=0 0 0 -> xyz=0.0849999999999993 0 0.0224999999279662 rpy=3.14159265358979 1.5707963267949 0
- joint leg_l4_joint: axis 0 1 0 -> 0 0 -1; limit lower=0 upper=1.5 effort=23.7 velocity=30.1 -> lower=-0.6806784082777885 upper=1.5707963267948966 effort=30 velocity=14; origin xyz=0 0.0145 -0.24 rpy=0 0 0 -> xyz=-0.119085999406409 -0.10231092202195 -0.00450000000000123 rpy=0 0 0
- joint leg_l5_fixed_1: child leg_l_f1_link -> leg_l_f2_link; origin xyz=0.06 0 -0.007 rpy=0 0 0 -> xyz=-0.094 0 -0.11 rpy=0 0 0
- joint leg_l5_fixed_2: child leg_l_f2_link -> leg_l_f1_link; origin xyz=-0.030 0 -0.007 rpy=0 0 0 -> xyz=0.1515 0 -0.11 rpy=0 0 0
- joint leg_l5_joint: limit lower=-1.1 upper=1.1 effort=23.7 velocity=30.1 -> lower=-0.5061454830783556 upper=1.064650843716541 effort=12 velocity=14; origin xyz=0.005 0 -0.23995 rpy=0 0 0 -> xyz=0.101882292521187 -0.109129160590203 -0.0445000000000359 rpy=-1.5707 0 0
- joint leg_r1_joint: axis 1 0 0 -> 0 0 1; limit lower=-0.5 upper=0.2 effort=23.7 velocity=30.1 -> lower=-0.34906 upper=0.34906 effort=12 velocity=14; origin xyz=-0.002 -0.09 -0.1035 rpy=0 0 0 -> xyz=0.0200750000000058 -0.0679999999999992 0.138 rpy=0 0 0
- joint leg_r2_joint: axis 0 0 1 -> 0 0 -1; limit lower=-1 upper=0.5 effort=23.7 velocity=30.1 -> lower=-0.17453 upper=0.34906 effort=12 velocity=14; origin xyz=0 0.00016972 -0.0325 rpy=0 0 0 -> xyz=0.0224999999999977 0 -0.0714999999999994 rpy=-1.57079632679488 0 1.5707963267949
- joint leg_r3_joint: axis 0 1 0 -> 0 0 -1; limit lower=-1.2 upper=0.8 effort=23.7 velocity=30.1 -> lower=-0.698131 upper=1.8 effort=12 velocity=14; origin xyz=0 0.01633 -0.0575 rpy=0 0 0 -> xyz=-0.0849999999999561 0 0.0224999999468524 rpy=0 1.5707963267949 0
- joint leg_r4_joint: axis 0 1 0 -> 0 0 1; limit lower=0 upper=1.5 effort=23.7 velocity=30.1 -> lower=-1.5707963 upper=0.680678 effort=30 velocity=14; origin xyz=0 -0.0145 -0.24 rpy=0 0 0 -> xyz=-0.114760457317049 0.107140270037781 -0.00450000000003428 rpy=3.14159265358979 0 0
- joint leg_r5_fixed_1: origin xyz=0.06 0 -0.007 rpy=0 0 0 -> xyz=0.1515 0 -0.11 rpy=0 0 0
- joint leg_r5_fixed_2: origin xyz=-0.030 0 -0.007 rpy=0 0 0 -> xyz=-0.094 0 -0.11 rpy=0 0 0
- joint leg_r5_joint: limit lower=-1.1 upper=1.1 effort=23.7 velocity=30.1 -> lower=-1.0646 upper=0.50614 effort=12 velocity=14; origin xyz=0.005 0 -0.23995 rpy=0 0 0 -> xyz=0.10199 -0.10903 0.0445 rpy=-1.5707 0 0

Commit message: feat:成功站立模型

File: src/hunter_bipedal_control/legged_examples/legged_hunter/legged_hunter_description/urdf/hunter.urdf (robot description, URDF)
Before this commit: robot tangba, 16 links, 15 joints
Links:
- link base_link: mass 9.2349183 -> 3.71439
- link leg_l4_link: geometry collision box size=0.12 0.1 0.06; visual mesh filename=package://legged_hunter_description/tangba_meshes/link_left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
- link leg_l5_link: geometry collision box size=0.1 0.08 0.15; visual mesh filename=package://legged_hunter_description/tangba_meshes/link_left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
- link leg_r4_link: geometry collision box size=0.12 0.1 0.06; visual mesh filename=package://legged_hunter_description/tangba_meshes/link_righ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
- link leg_r5_link: geometry collision box size=0.1 0.08 0.15; visual mesh filename=package://legged_hunter_description/tangba_meshes/link_righ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

Commit message: feat:步态优化

File: src/hunter_bipedal_control/legged_examples/legged_hunter/legged_hunter_description/urdf/hunter.urdf (robot description, URDF)
Before this commit: robot tangba, 16 links, 15 joints
Links:
- link leg_l5_link: geometry collision box size=0.2 0.08 0.15; visual mesh filename=package://legged_hunter_description/tangba_meshes/link_left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
- link leg_r5_link: geometry collision box size=0.2 0.08 0.15; visual mesh filename=package://legged_hunter_description/tangba_meshes/link_righ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

Commit message: fix:调整步态

File: src/hunter_bipedal_control/legged_examples/legged_hunter/legged_hunter_description/urdf/hunter.urdf (robot description, URDF)
Before this commit: robot tangba, 16 links, 15 joints
Links:
- link leg_l3_link: geometry collision box size=0.12 0.1 0.06; visual mesh filename=package://legged_hunter_description/tangba_meshes/link_left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
- link leg_l5_link: geometry collision box size=0.23 0.08 0.15; visual mesh filename=package://legged_hunter_description/tangba_meshes/link_left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
- link leg_r3_link: geometry collision box size=0.12 0.1 0.06; visual mesh filename=package://legged_hunter_description/tangba_meshes/link_righ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
- link leg_r5_link: geometry collision box size=0.23 0.08 0.15; visual mesh filename=package://legged_hunter_description/tangba_meshes/link_righ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
Joints:
- joint leg_l5_fixed_1: child leg_l_f2_link -> leg_l_f1_link; origin xyz=-0.094 0 -0.11 rpy=0 0 0 -> xyz=0.1515 0 -0.11 rpy=0 0 0
- joint leg_l5_fixed_2: child leg_l_f1_link -> leg_l_f2_link; origin xyz=0.1515 0 -0.11 rpy=0 0 0 -> xyz=-0.094 0 -0.11 rpy=0 0 0

Commit message: feat:增加原始task,修改urdf参数

File: src/hunter_bipedal_control/legged_examples/legged_hunter/legged_hunter_description/urdf/hunter.urdf (robot description, URDF)
Before this commit: robot tangba, 16 links, 15 joints
Joints:
- joint leg_l5_fixed_1: origin xyz=0.1515 0 -0.11 rpy=0 0 0 -> xyz=0.1515 -0.031 -0.11 rpy=0 0 0
- joint leg_l5_fixed_2: origin xyz=-0.094 0 -0.11 rpy=0 0 0 -> xyz=-0.094 -0.031 -0.11 rpy=0 0 0
- joint leg_r5_fixed_1: origin xyz=0.1515 0 -0.11 rpy=0 0 0 -> xyz=0.1515 0.031 -0.11 rpy=0 0 0
- joint leg_r5_fixed_2: origin xyz=-0.094 0 -0.11 rpy=0 0 0 -> xyz=-0.094 0.031 -0.11 rpy=0 0 0
